Commit message: removed unnecessary code and alined camera with robot model

File: src/moma_visualisation/urdf/robot.urdf.xacro (robot description, xacro)
@@ -28,7 +28,7 @@
     </joint>
     <joint name="camera_joint" type="fixed">
-        <parent link="link_6"/>
+        <parent link="flange"/>
         <child link="camera_link"/>
-        <origin xyz="0.305 0 0.08" rpy="0 0 0"/>
+        <origin xyz="0 0.08 0.05" rpy="0 -1.5707 0"/>
     </joint>
     <link name="camera_link">

Commit message: Fixed camera orientation

File: src/moma_visualisation/urdf/robot.urdf.xacro (robot description, xacro)
@@ -30,5 +30,5 @@
         <parent link="flange"/>
         <child link="camera_link"/>
-        <origin xyz="0 0.08 0.05" rpy="0 -1.5707 0"/>
+        <origin xyz="0 0.08 0.05" rpy="-1.5707 -1.5707 0"/>
     </joint>
     <link name="camera_link">
