Commit message: camera

File: src/moma_visualisation/urdf/macro.gazebo.xacro (robot description, xacro)
@@ -20,4 +20,57 @@
       <self_collide>true</self_collide>
     </gazebo>
+    <gazebo reference="camera_link">
+      <material>Gazebo/Red</material>
+      <sensor name="camera1" type="camera">
+        <pose> 0 0 0 0 0 0 </pose>
+        <update_rate>10</update_rate>
+        <frame_id>base_camera</frame_id>
+        <topic>/test/integration/CameraPlugin_imagesWithBuiltinSDF</topic>
+        <camera>
+          <horizontal_fov>1.05</horizontal_fov>
+          <image>
+            <width>256</width>
+            <height>257</height>
+          </image>
+          <clip>
+            <near>0.1</near>
+            <far>10.0</far>
+          </clip>
+          <noise>
+            <type>gaussian</type>
+            <mean>0.0</mean>
+            <stddev>0.007</stddev>
+          </noise>
+          <lens>
+            <type>custom</type>
+            <scale_to_hfov>false</scale_to_hfov>
+            <custom_function>
+              <c1>1.1</c1>
+              <c2>2.2</c2>
+              <c3>3.3</c3>
+              <f>1.2</f>
+              <fun>sin</fun>
+            </custom_function>
+            <cutoff_angle>0.7505</cutoff_angle>
+            <env_texture_size>128</env_texture_size>
+            <intrinsics>
+              <fx>280</fx>
+              <fy>281</fy>
+              <cx>162</cx>
+              <cy>124</cy>
+              <s>1.2</s>
+            </intrinsics>
+            <projection>
+              <p_fx>282</p_fx>
+              <p_fy>283</p_fy>
+              <p_cx>163</p_cx>
+              <p_cy>125</p_cy>
+              <tx>1</tx>
+              <ty>2</ty>
+            </projection>
+          </lens>
+        </camera>
+      </sensor>
+    </gazebo>
   </xacro:macro>
 </robot>

File: src/moma_visualisation/urdf/robot.urdf.xacro (robot description, xacro)
@@ -27,4 +27,17 @@
         <origin xyz="0 0 0" rpy="0 0 0" />
     </joint>
+    <joint name="camera_joint" type="fixed">
+        <parent link="link_6"/>
+        <child link="camera_link"/>
+        <origin xyz="0.305 0 0.08" rpy="0 0 0"/>
+    </joint>
+    <link name="camera_link">
+        <visual>
+            <geometry>
+                <box size="0.010 0.03 0.03"/>
+            </geometry>
+            <material name="red"/>
+        </visual>
+    </link>
     <xacro:include filename="gazebo_control.xacro"/>
 </robot>

Commit message: depth camera working

File: src/moma_visualisation/urdf/macro.gazebo.xacro (robot description, xacro)
@@ -20,55 +20,52 @@
       <self_collide>true</self_collide>
     </gazebo>
-    <gazebo reference="camera_link">
-      <material>Gazebo/Red</material>
-      <sensor name="camera1" type="camera">
-        <pose> 0 0 0 0 0 0 </pose>
-        <update_rate>10</update_rate>
-        <frame_id>base_camera</frame_id>
-        <topic>/test/integration/CameraPlugin_imagesWithBuiltinSDF</topic>
-        <camera>
-          <horizontal_fov>1.05</horizontal_fov>
+    <gazebo reference="${prefix}camera_link">
+      <sensor name="rgbd_camera" type="rgbd_camera">
+        <ignition_frame_id>${prefix}camera_link</ignition_frame_id>
+        <frame_id>${prefix}camera_link</frame_id>
+        <camera name="rgbd_camera_frame">
+          <horizontal_fov>1.3962634</horizontal_fov>
+          <lens>
+            <intrinsics>
+              <fx>277.1</fx>
+              <fy>277.1</fy>
+              <cx>160.5</cx>
+              <cy>120.5</cy>
+              <s>0</s>
+            </intrinsics>
+          </lens>
+          <distortion>
+            <k1>0.104207</k1>
+            <k2>-0.255558</k2>
+            <k3>0.128694</k3>
+            <p1>0.000512</p1>
+            <p2>0.000319</p2>
+            <center>0.5 0.5</center>
+          </distortion>
           <image>
-            <width>256</width>
-            <height>257</height>
+            <width>1280</width>
+            <height>720</height>
+            <format>L8</format>
           </image>
           <clip>
-            <near>0.1</near>
-            <far>10.0</far>
+            <near>0.01</near>
+            <far>300</far>
           </clip>
+          <depth_camera>
+            <clip>
+              <near>0.1</near>
+              <far>10</far>
+            </clip>
+          </depth_camera>
           <noise>
             <type>gaussian</type>
-            <mean>0.0</mean>
-            <stddev>0.007</stddev>
+            <mean>0</mean>
+            <stddev>0.003</stddev>
           </noise>
-          <lens>
-            <type>custom</type>
-            <scale_to_hfov>false</scale_to_hfov>
-            <custom_function>
-              <c1>1.1</c1>
-              <c2>2.2</c2>
-              <c3>3.3</c3>
-              <f>1.2</f>
-              <fun>sin</fun>
-            </custom_function>
-            <cutoff_angle>0.7505</cutoff_angle>
-            <env_texture_size>128</env_texture_size>
-            <intrinsics>
-              <fx>280</fx>
-              <fy>281</fy>
-              <cx>162</cx>
-              <cy>124</cy>
-              <s>1.2</s>
-            </intrinsics>
-            <projection>
-              <p_fx>282</p_fx>
-              <p_fy>283</p_fy>
-              <p_cx>163</p_cx>
-              <p_cy>125</p_cy>
-              <tx>1</tx>
-              <ty>2</ty>
-            </projection>
-          </lens>
         </camera>
+        <always_on>1</always_on>
+        <update_rate>10</update_rate>
+        <visualize>0</visualize>
+        <topic>depth_camera</topic>
       </sensor>
     </gazebo>

File: src/moma_visualisation/urdf/macro.tm12s-nominal.urdf.xacro (robot description, xacro)
@@ -327,4 +327,19 @@
       </inertial>
     </link>
+    <!-- RGBD Camera -->
+    <joint name="camera_joint" type="fixed">
+        <parent link="${prefix}link_6"/>
+        <child link="${prefix}camera_link"/>
+        <origin xyz="0 0.08 0.05" rpy="-1.5707 -1.5707 0"/>
+    </joint>
+    <link name="${prefix}camera_link">
+        <visual>
+            <geometry>
+                <box size="0.010 0.03 0.03"/>
+            </geometry>
+            <material name="red"/>
+        </visual>
+        <static>true</static>
+    </link>
     <link name="${prefix}flange" />
     <!-- Joint -->

File: src/moma_visualisation/urdf/robot.urdf.xacro (robot description, xacro)
@@ -27,17 +27,4 @@
         <origin xyz="0 0 0" rpy="0 0 0" />
     </joint>
-    <joint name="camera_joint" type="fixed">
-        <parent link="flange"/>
-        <child link="camera_link"/>
-        <origin xyz="0 0.08 0.05" rpy="-1.5707 -1.5707 0"/>
-    </joint>
-    <link name="camera_link">
-        <visual>
-            <geometry>
-                <box size="0.010 0.03 0.03"/>
-            </geometry>
-            <material name="red"/>
-        </visual>
-    </link>
     <xacro:include filename="gazebo_control.xacro"/>
 </robot>
