Commit message: massive update: gazebo sim, moveit, nav2 everything working simultaneously YOLO not working

File: src/moma_visualisation/urdf/gazebo_control.xacro (robot description, xacro)
@@ -107,4 +107,33 @@
       <state_interface name="velocity"/>
     </joint>
+    <joint name="finger_joint">
+      <command_interface name="position" />
+      <state_interface name="position">
+        <param name="initial_value">0.05</param>
+      </state_interface>
+      <state_interface name="velocity">
+        <param name="initial_value">0.0</param>
+      </state_interface>
+    </joint>
+    <joint name="left_inner_knuckle_joint">
+      <param name="mimic">finger_joint</param>
+      <param name="multiplier">-1</param>
+    </joint>
+    <joint name="left_inner_finger_joint">
+      <param name="mimic">finger_joint</param>
+      <param name="multiplier">1</param>
+    </joint>
+    <joint name="right_outer_knuckle_joint">
+      <param name="mimic">finger_joint</param>
+      <param name="multiplier">-1</param>
+    </joint>
+    <joint name="right_inner_knuckle_joint">
+      <param name="mimic">finger_joint</param>
+      <param name="multiplier">-1</param>
+    </joint>
+    <joint name="right_inner_finger_joint">
+      <param name="mimic">finger_joint</param>
+      <param name="multiplier">1</param>
+    </joint>
   </ros2_control>
   <gazebo>

File: src/moma_visualisation/urdf/macro.tm12s-nominal.urdf.xacro (robot description, xacro)
@@ -350,4 +350,43 @@
     </joint>
     <!--LinkDescription-->
+    <!-- <xacro:include filename="$(find moma_visualisation)/urdf/2f_140.ros2_control.xacro" /> -->
+    <joint name="${prefix}robotiq_base_joint" type="fixed">
+      <parent link="${prefix}flange" />
+      <child link="${prefix}robotiq_140_base_link" />
+      <origin xyz="0 0 0" rpy="0 0 ${pi/2}" />
+    </joint>
+    <link name="${prefix}robotiq_140_base_link">
+      <inertial>
+        <origin xyz="8.625E-08 -4.6583E-06 0.03145" rpy="0 0 0" />
+        <mass value="0.22652" />
+        <inertia ixx="0.00020005" ixy="-4.2442E-10" ixz="-2.9069E-10" iyy="0.00017832" iyz="-3.4402E-08" izz="0.00013478" />
+      </inertial>
+      <visual>
+        <origin xyz="0 0 0" rpy="0 0 0" />
+        <geometry>
+          <mesh filename="file://$(find moma_visualisation)/meshes/robotiq_2f_140_base_link.stl" />
+        </geometry>
+        <material name="">
+          <color rgba="0.1 0.1 0.1 1" />
+        </material>
+      </visual>
+      <collision>
+        <origin xyz="0 0 0" rpy="0 0 0" />
+        <geometry>
+          <mesh filename="file://$(find moma_visualisation)/meshes/robotiq_2f_140_base_link.stl" />
+        </geometry>
+      </collision>
+    </link>
+  <!-- <joint name="${prefix}robotiq_140_base_joint" type="fixed">
+      <parent link="${prefix}robotiq_base_link" />
+      <child link="${prefix}robotiq_140_base_link" />
+      <xacro:insert_block name="origin" />
+  </joint> -->
+  <!-- Include the finger xacros and run them -->
+  <xacro:include filename="$(find moma_visualisation)/urdf/robotiq_2f_140.xacro" />
+  <xacro:finger_links prefix="${prefix}" fingerprefix="left" stroke="140"/>
+  <xacro:finger_links prefix="${prefix}" fingerprefix="right" stroke="140"/>
+  <xacro:finger_joint prefix="${prefix}"/>
+  <xacro:right_outer_knuckle_joint prefix="${prefix}"/>
   </xacro:macro>
 </robot>
