Commit message: robot movements and stuff working, now with LD250 instead of 90

File: src/moma_visualisation/urdf/amr_core.xacro (robot description, xacro)
@@ -2,4 +2,5 @@
 <robot name="AMR_Platform"
   xmlns:xacro="http://www.ros.org/wiki/xacro">
+  <!-- COLOURS -->
   <material name="amr_body_color">
     <color rgba="0.5 0.4 0.9 1.0"/>
@@ -12,6 +13,7 @@
     <static>true</static>
   </link>
+  <!-- MAIN BODY COMPOSED OF 3 ABSTRACT BOXES -->
   <link name="amr_main_body">
-    <visual>
+    <!-- <visual>
       <origin rpy="0 0 0" xyz="0 0 0.01"/>
       <geometry>
@@ -33,6 +35,12 @@
       </geometry>
       <material name="amr_body_color"></material>
-    </visual>
-    <!--  -->
+    </visual> -->
+    <visual>
+      <origin rpy="0 0 3.1415926535897" xyz="0 0 -0.085"/>
+      <geometry>
+        <mesh filename="package://moma_visualisation/meshes/LD250.obj"/>
+      </geometry>
+      <material name="white"/>
+    </visual>
     <collision>
       <origin rpy="0 0 0" xyz="0 0 0.01"/>
@@ -53,6 +61,18 @@
       </geometry>
     </collision>
-    <inertial>
+    <!-- <collision>
+      <origin rpy="1.5707963267949 0 1.5707963267949" xyz="0 0 0"/>
+      <geometry>
+        <mesh filename="package://moma_visualisation/meshes/AMR_Platform.STL"/>
+      </geometry>
+    </collision> -->
+    <!-- <inertial>
       <mass value="10000.07"/>
+      <origin rpy="0 0 0" xyz="-0.03 0 0"/>
+      <inertia ixx="0.426" ixy="0.0" ixz="0.0" iyy="0.496" iyz="0.0" izz="0.91"/>
+    </inertial> -->
+    <inertial>
+      <!-- <mass value="4.07"/> -->
+      <mass value="146"/> <!-- TRUE MASS FROM DATASHEET -->
       <origin rpy="0 0 0" xyz="-0.03 0 0"/>
       <inertia ixx="0.426" ixy="0.0" ixz="0.0" iyy="0.496" iyz="0.0" izz="0.91"/>
@@ -68,12 +88,12 @@
       <origin rpy="1.5707963267949 0 0" xyz="0 0 0"/>
       <geometry>
-        <cylinder length="0.03937" radius="0.088"/>
-      </geometry>
-      <material name="amr_wheel_color"/>
-    </visual>
-    <collision>
-      <origin rpy="1.5707963267949 0 0" xyz="0 0 0"/>
-      <geometry>
-        <cylinder length="0.03937" radius="0.088"/>
+        <cylinder length="0.03937" radius="0.105"/>
+      </geometry>
+      <material name="amr_wheel_color"/>
+    </visual>
+    <collision>
+      <origin rpy="1.5707963267949 0 0" xyz="0 0 0"/>
+      <geometry>
+        <cylinder length="0.03937" radius="0.105"/>
       </geometry>
     </collision>
@@ -87,5 +107,6 @@
     <parent link="amr_main_body"/>
     <child link="left_wheel"/>
-    <origin rpy="0 0 0" xyz="0 0.3 0.000881"/>
+    <!-- <origin rpy="0 0 0" xyz="0 0.3 0.000881"/> -->
+    <origin rpy="0 0 0" xyz="-0.004 0.3025 0.02"/>
   </joint>
   <link name="right_wheel">
@@ -93,12 +114,12 @@
       <origin rpy="1.5707963267949 0 0" xyz="0 0 0"/>
       <geometry>
-        <cylinder length="0.03937" radius="0.088"/>
-      </geometry>
-      <material name="amr_wheel_color"/>
-    </visual>
-    <collision>
-      <origin rpy="1.5707963267949 0 0" xyz="0 0 0"/>
-      <geometry>
-        <cylinder length="0.03937" radius="0.088"/>
+        <cylinder length="0.03937" radius="0.105"/>
+      </geometry>
+      <material name="amr_wheel_color"/>
+    </visual>
+    <collision>
+      <origin rpy="1.5707963267949 0 0" xyz="0 0 0"/>
+      <geometry>
+        <cylinder length="0.03937" radius="0.105"/>
       </geometry>
     </collision>
@@ -112,5 +133,6 @@
     <parent link="amr_main_body"/>
     <child link="right_wheel"/>
-    <origin rpy="0 0 0" xyz="0 -0.3 0.000881"/>
+    <!-- <origin rpy="0 0 0" xyz="0 -0.3 0.000881"/> -->
+    <origin rpy="0 0 0" xyz="-0.004 -0.3025 0.02"/>
   </joint>
   <link name="right_front_small_wheel">
@@ -118,12 +140,12 @@
       <origin rpy="1.5707963267949 0 0" xyz="0 0 0"/>
       <geometry>
-        <cylinder length="0.02775" radius="0.03625"/>
-      </geometry>
-      <material name="amr_wheel_color"/>
-    </visual>
-    <collision>
-      <origin rpy="1.5707963267949 0 0" xyz="0 0 0"/>
-      <geometry>
-        <cylinder length="0.02775" radius="0.03625"/>
+        <cylinder length="0.02775" radius="0.063"/>
+      </geometry>
+      <material name="amr_wheel_color"/>
+    </visual>
+    <collision>
+      <origin rpy="1.5707963267949 0 0" xyz="0 0 0"/>
+      <geometry>
+        <cylinder length="0.02775" radius="0.063"/>
       </geometry>
     </collision>
@@ -137,5 +159,5 @@
     <parent link="amr_main_body"/>
     <child link="right_front_small_wheel"/>
-    <origin rpy="0 0 0" xyz="0.209 -0.108 -0.049"/>
+    <origin rpy="0 0 0" xyz="0.2493 -0.2325 -0.022"/>
   </joint>
   <link name="left_front_small_wheel">
@@ -143,12 +165,12 @@
       <origin rpy="1.5707963267949 0 0" xyz="0 0 0"/>
       <geometry>
-        <cylinder length="0.02775" radius="0.03625"/>
-      </geometry>
-      <material name="amr_wheel_color"/>
-    </visual>
-    <collision>
-      <origin rpy="1.5707963267949 0 0" xyz="0 0 0"/>
-      <geometry>
-        <cylinder length="0.02775" radius="0.03625"/>
+        <cylinder length="0.02775" radius="0.063"/>
+      </geometry>
+      <material name="amr_wheel_color"/>
+    </visual>
+    <collision>
+      <origin rpy="1.5707963267949 0 0" xyz="0 0 0"/>
+      <geometry>
+        <cylinder length="0.02775" radius="0.063"/>
       </geometry>
     </collision>
@@ -162,5 +184,5 @@
     <parent link="amr_main_body"/>
     <child link="left_front_small_wheel"/>
-    <origin rpy="0 0 0" xyz="0.209 0.108 -0.049"/>
+    <origin rpy="0 0 0" xyz="0.2493 0.2325 -0.022"/>
   </joint>
   <link name="left_back_small_wheel">
@@ -168,12 +190,12 @@
       <origin rpy="1.5707963267949 0 0" xyz="0 0 0"/>
       <geometry>
-        <cylinder length="0.02775" radius="0.03625"/>
-      </geometry>
-      <material name="amr_wheel_color"/>
-    </visual>
-    <collision>
-      <origin rpy="1.5707963267949 0 0" xyz="0 0 0"/>
-      <geometry>
-        <cylinder length="0.02775" radius="0.03625"/>
+        <cylinder length="0.02775" radius="0.063"/>
+      </geometry>
+      <material name="amr_wheel_color"/>
+    </visual>
+    <collision>
+      <origin rpy="1.5707963267949 0 0" xyz="0 0 0"/>
+      <geometry>
+        <cylinder length="0.02775" radius="0.063"/>
       </geometry>
     </collision>
@@ -187,5 +209,5 @@
     <parent link="amr_main_body"/>
     <child link="left_back_small_wheel"/>
-    <origin rpy="0 0 0" xyz="-0.228 0.156 -0.049"/>
+    <origin rpy="0 0 0" xyz="-0.257 0.2325 -0.022"/>
   </joint>
   <link name="right_back_small_wheel">
@@ -193,12 +215,12 @@
       <origin rpy="1.5707963267949 0 0" xyz="0 0 0"/>
       <geometry>
-        <cylinder length="0.02775" radius="0.03625"/>
-      </geometry>
-      <material name="amr_wheel_color"/>
-    </visual>
-    <collision>
-      <origin rpy="1.5707963267949 0 0" xyz="0 0 0"/>
-      <geometry>
-        <cylinder length="0.02775" radius="0.03625"/>
+        <cylinder length="0.02775" radius="0.063"/>
+      </geometry>
+      <material name="amr_wheel_color"/>
+    </visual>
+    <collision>
+      <origin rpy="1.5707963267949 0 0" xyz="0 0 0"/>
+      <geometry>
+        <cylinder length="0.02775" radius="0.063"/>
       </geometry>
     </collision>
@@ -212,5 +234,5 @@
     <parent link="amr_main_body"/>
     <child link="right_back_small_wheel"/>
-    <origin rpy="0 0 0" xyz="-0.228 -0.156 -0.049"/>
+    <origin rpy="0 0 0" xyz="-0.257 -0.2325 -0.022"/>
   </joint>
 </robot>

File: src/moma_visualisation/urdf/amr_lidar.xacro (robot description, xacro)
@@ -17,5 +17,5 @@
         <visual>
             <geometry>
-                <cylinder length="0.004" radius="0.007"/>
+                <cylinder length="0.050" radius="0.050"/>
             </geometry>
             <material name="amr_laser_red"/>

File: src/moma_visualisation/urdf/chassis_core.xacro (robot description, xacro)
@@ -6,8 +6,8 @@
       <origin rpy="0 0 0" xyz="0 0 0.545"/>
       <geometry>
-        <box size="0.8 0.69 0.35 "/>
+        <box size="0.95 0.69 0.35 "/>
       </geometry>
     </visual>
-    <visual>
+    <!-- <visual>
       <material name="amr_body_color" />
       <origin rpy="0 0 0" xyz="-0.1 -0.31 0.17"/>
@@ -22,12 +22,12 @@
         <box size="0.6 0.04 0.38 "/>
       </geometry>
-    </visual>
+    </visual> -->
     <collision>
       <origin rpy="0 0 0" xyz="0 0 0.545"/>
       <geometry>
-        <box size="0.8 0.69 0.35 "/>
+        <box size="0.95 0.69 0.35 "/>
       </geometry>
     </collision>
-    <collision>
+    <!-- <collision>
       <origin rpy="0 0 0" xyz="-0.1 -0.31 0.17"/>
       <geometry>
@@ -40,5 +40,5 @@
         <box size="0.6 0.04 0.38 "/>
       </geometry>
-    </collision>
+    </collision> -->
   </link>
 </robot>

File: src/moma_visualisation/urdf/robot.urdf.xacro (robot description, xacro)
@@ -8,5 +8,6 @@
         <parent link="amr_main_body"/>
         <child link="amr_lidar_body"/>
-        <origin xyz="0.35 0 0.1"/>
+        <!-- <origin xyz="0.35 0 0.1"/> -->
+        <origin xyz="0.35 0 0.115"/>
     </joint>
     <joint name="chassis_connector" type="fixed">

File: src/moma_visualisation/urdf/tm12s_core.xacro (robot description, xacro)
@@ -5,5 +5,4 @@
   <xacro:arg name="color" default="darkolive" />
   <xacro:arg name="trans_hw_iface" default="hardware_interface/PositionJointInterface" />
-  <xacro:include filename="macro.gazebo.xacro" />
   <xacro:include filename="macro.transmission.xacro" />
   <xacro:include filename="macro.materials.xacro" />
@@ -12,4 +11,5 @@
   <!-- you must modify 'macro.tm12s-nominal.urdf.xacro' to 'user_defined.urdf.xacro'  -->
   <xacro:include filename="macro.tm12s-nominal.urdf.xacro" />
+  <xacro:include filename="macro.gazebo.xacro" />
   <!--  -->
   <xacro:tmr_gazebo ns="$(arg ns)" prefix="$(arg prefix)" />

Commit message: both working but nav2 overestimating in rviz

File: src/moma_visualisation/urdf/amr_core.xacro (robot description, xacro)
@@ -15,26 +15,33 @@
   <!-- MAIN BODY COMPOSED OF 3 ABSTRACT BOXES -->
   <link name="amr_main_body">
+    <visual>
+      <origin rpy="0 0 0" xyz="0 0 0.01"/>
+      <geometry>
+        <box size="0.7 0.5 0.14 "/>
+      </geometry>
+      <material name="amr_body_color"></material>
+    </visual>
+    <visual>
+      <origin rpy="0 0 0" xyz="-0.125 0 0.11"/>
+      <geometry>
+        <box size="0.45 0.5 0.05 "/>
+      </geometry>
+      <material name="amr_body_color"></material>
+    </visual>
+    <visual>
+      <origin rpy="0 0 0" xyz="0 0 0.21"/>
+      <geometry>
+        <box size="0.7 0.5 0.14 "/>
+      </geometry>
+      <material name="amr_body_color"></material>
+    </visual>
     <!-- <visual>
-      <origin rpy="0 0 0" xyz="0 0 0.01"/>
-      <geometry>
-        <box size="0.7 0.5 0.14 "/>
-      </geometry>
-      <material name="amr_body_color"></material>
-    </visual>
-    <visual>
-      <origin rpy="0 0 0" xyz="-0.125 0 0.11"/>
-      <geometry>
-        <box size="0.45 0.5 0.05 "/>
-      </geometry>
-      <material name="amr_body_color"></material>
-    </visual>
-    <visual>
-      <origin rpy="0 0 0" xyz="0 0 0.21"/>
-      <geometry>
-        <box size="0.7 0.5 0.14 "/>
-      </geometry>
-      <material name="amr_body_color"></material>
+      <origin rpy="-1.5707963267949 0 3.1415926535897" xyz="0 0 -0.085"/>
+      <geometry>
+        <mesh filename="package://moma_visualisation/meshes/amr_chassis_scaled.stl"/>
+      </geometry>
+      <material name="white"/>
     </visual> -->
-    <visual>
+    <!-- <visual>
       <origin rpy="0 0 3.1415926535897" xyz="0 0 -0.085"/>
       <geometry>
@@ -42,5 +49,5 @@
       </geometry>
       <material name="white"/>
-    </visual>
+    </visual> -->
     <collision>
       <origin rpy="0 0 0" xyz="0 0 0.01"/>
@@ -64,5 +71,5 @@
       <origin rpy="1.5707963267949 0 1.5707963267949" xyz="0 0 0"/>
       <geometry>
-        <mesh filename="package://moma_visualisation/meshes/AMR_Platform.STL"/>
+        <mesh filename="package://moma_visualisation/meshes/LD250.obj"/>
       </geometry>
     </collision> -->
@@ -74,5 +81,5 @@
     <inertial>
       <!-- <mass value="4.07"/> -->
-      <mass value="146"/> <!-- TRUE MASS FROM DATASHEET -->
+      <mass value="10000.07"/> <!-- TRUE MASS FROM DATASHEET + 60 -->
       <origin rpy="0 0 0" xyz="-0.03 0 0"/>
       <inertia ixx="0.426" ixy="0.0" ixz="0.0" iyy="0.496" iyz="0.0" izz="0.91"/>
@@ -82,5 +89,5 @@
     <parent link="base_link"/>
     <child link="amr_main_body"/>
-    <origin xyz="0 0 0.09"/>
+    <origin xyz="0 0 0.15"/>
   </joint>
   <link name="left_wheel">

File: src/moma_visualisation/urdf/chassis_core.xacro (robot description, xacro)
@@ -4,7 +4,7 @@
     <visual>
       <material name="amr_body_color" />
-      <origin rpy="0 0 0" xyz="0 0 0.545"/>
+      <origin rpy="0 0 0" xyz="0.078 0 0.545"/>
       <geometry>
-        <box size="0.95 0.69 0.35 "/>
+        <box size="0.95 0.7 0.37 "/>
       </geometry>
     </visual>
@@ -24,7 +24,7 @@
     </visual> -->
     <collision>
-      <origin rpy="0 0 0" xyz="0 0 0.545"/>
+      <origin rpy="0 0 0" xyz="0.078 0 0.545"/>
       <geometry>
-        <box size="0.95 0.69 0.35 "/>
+        <box size="0.95 0.7 0.37 "/>
       </geometry>
     </collision>

File: src/moma_visualisation/urdf/robot.urdf.xacro (robot description, xacro)
@@ -15,4 +15,5 @@
         <parent link="amr_main_body"/>
         <child link="chassis"/>
+        <origin xyz="-0.08 0 -0.07" rpy="0 0 0"/>
     </joint>
     <joint name="tm12s_base_fixed_joint" type="fixed">

Commit message: fixed nav

File: src/moma_visualisation/urdf/amr_core.xacro (robot description, xacro)
@@ -15,5 +15,5 @@
   <!-- MAIN BODY COMPOSED OF 3 ABSTRACT BOXES -->
   <link name="amr_main_body">
-    <visual>
+    <!-- <visual>
       <origin rpy="0 0 0" xyz="0 0 0.01"/>
       <geometry>
@@ -35,5 +35,5 @@
       </geometry>
       <material name="amr_body_color"></material>
-    </visual>
+    </visual> -->
     <!-- <visual>
       <origin rpy="-1.5707963267949 0 3.1415926535897" xyz="0 0 -0.085"/>
@@ -43,5 +43,5 @@
       <material name="white"/>
     </visual> -->
-    <!-- <visual>
+    <visual>
       <origin rpy="0 0 3.1415926535897" xyz="0 0 -0.085"/>
       <geometry>
@@ -49,5 +49,5 @@
       </geometry>
       <material name="white"/>
-    </visual> -->
+    </visual>
     <collision>
       <origin rpy="0 0 0" xyz="0 0 0.01"/>
@@ -80,6 +80,5 @@
     </inertial> -->
     <inertial>
-      <!-- <mass value="4.07"/> -->
-      <mass value="10000.07"/> <!-- TRUE MASS FROM DATASHEET + 60 -->
+      <mass value="10000.07"/>
       <origin rpy="0 0 0" xyz="-0.03 0 0"/>
       <inertia ixx="0.426" ixy="0.0" ixz="0.0" iyy="0.496" iyz="0.0" izz="0.91"/>
@@ -95,12 +94,12 @@
       <origin rpy="1.5707963267949 0 0" xyz="0 0 0"/>
       <geometry>
-        <cylinder length="0.03937" radius="0.105"/>
-      </geometry>
-      <material name="amr_wheel_color"/>
-    </visual>
-    <collision>
-      <origin rpy="1.5707963267949 0 0" xyz="0 0 0"/>
-      <geometry>
-        <cylinder length="0.03937" radius="0.105"/>
+        <cylinder length="0.03937" radius="0.088"/>
+      </geometry>
+      <material name="amr_wheel_color"/>
+    </visual>
+    <collision>
+      <origin rpy="1.5707963267949 0 0" xyz="0 0 0"/>
+      <geometry>
+        <cylinder length="0.03937" radius="0.088"/>
       </geometry>
     </collision>
@@ -115,5 +114,5 @@
     <child link="left_wheel"/>
     <!-- <origin rpy="0 0 0" xyz="0 0.3 0.000881"/> -->
-    <origin rpy="0 0 0" xyz="-0.004 0.3025 0.02"/>
+    <origin rpy="0 0 0" xyz="-0.004 0.3025 0.000881"/>
   </joint>
   <link name="right_wheel">
@@ -121,12 +120,12 @@
       <origin rpy="1.5707963267949 0 0" xyz="0 0 0"/>
       <geometry>
-        <cylinder length="0.03937" radius="0.105"/>
-      </geometry>
-      <material name="amr_wheel_color"/>
-    </visual>
-    <collision>
-      <origin rpy="1.5707963267949 0 0" xyz="0 0 0"/>
-      <geometry>
-        <cylinder length="0.03937" radius="0.105"/>
+        <cylinder length="0.03937" radius="0.088"/>
+      </geometry>
+      <material name="amr_wheel_color"/>
+    </visual>
+    <collision>
+      <origin rpy="1.5707963267949 0 0" xyz="0 0 0"/>
+      <geometry>
+        <cylinder length="0.03937" radius="0.088"/>
       </geometry>
     </collision>
@@ -141,5 +140,5 @@
     <child link="right_wheel"/>
     <!-- <origin rpy="0 0 0" xyz="0 -0.3 0.000881"/> -->
-    <origin rpy="0 0 0" xyz="-0.004 -0.3025 0.02"/>
+    <origin rpy="0 0 0" xyz="-0.004 -0.3025 0.000881"/>
   </joint>
   <link name="right_front_small_wheel">
@@ -147,12 +146,12 @@
       <origin rpy="1.5707963267949 0 0" xyz="0 0 0"/>
       <geometry>
-        <cylinder length="0.02775" radius="0.063"/>
-      </geometry>
-      <material name="amr_wheel_color"/>
-    </visual>
-    <collision>
-      <origin rpy="1.5707963267949 0 0" xyz="0 0 0"/>
-      <geometry>
-        <cylinder length="0.02775" radius="0.063"/>
+        <cylinder length="0.02775" radius="0.03625"/>
+      </geometry>
+      <material name="amr_wheel_color"/>
+    </visual>
+    <collision>
+      <origin rpy="1.5707963267949 0 0" xyz="0 0 0"/>
+      <geometry>
+        <cylinder length="0.02775" radius="0.03625"/>
       </geometry>
     </collision>
@@ -166,5 +165,6 @@
     <parent link="amr_main_body"/>
     <child link="right_front_small_wheel"/>
-    <origin rpy="0 0 0" xyz="0.2493 -0.2325 -0.022"/>
+    <!-- <origin rpy="0 0 0" xyz="0.209 -0.108 -0.049"/> -->
+    <origin rpy="0 0 0" xyz="0.2493 -0.2325 -0.049"/>
   </joint>
   <link name="left_front_small_wheel">
@@ -172,12 +172,12 @@
       <origin rpy="1.5707963267949 0 0" xyz="0 0 0"/>
       <geometry>
-        <cylinder length="0.02775" radius="0.063"/>
-      </geometry>
-      <material name="amr_wheel_color"/>
-    </visual>
-    <collision>
-      <origin rpy="1.5707963267949 0 0" xyz="0 0 0"/>
-      <geometry>
-        <cylinder length="0.02775" radius="0.063"/>
+        <cylinder length="0.02775" radius="0.03625"/>
+      </geometry>
+      <material name="amr_wheel_color"/>
+    </visual>
+    <collision>
+      <origin rpy="1.5707963267949 0 0" xyz="0 0 0"/>
+      <geometry>
+        <cylinder length="0.02775" radius="0.03625"/>
       </geometry>
     </collision>
@@ -191,5 +191,6 @@
     <parent link="amr_main_body"/>
     <child link="left_front_small_wheel"/>
-    <origin rpy="0 0 0" xyz="0.2493 0.2325 -0.022"/>
+    <!-- <origin rpy="0 0 0" xyz="0.209 0.108 -0.049"/> -->
+    <origin rpy="0 0 0" xyz="0.2493 0.2325 -0.049"/>
   </joint>
   <link name="left_back_small_wheel">
@@ -197,12 +198,12 @@
       <origin rpy="1.5707963267949 0 0" xyz="0 0 0"/>
       <geometry>
-        <cylinder length="0.02775" radius="0.063"/>
-      </geometry>
-      <material name="amr_wheel_color"/>
-    </visual>
-    <collision>
-      <origin rpy="1.5707963267949 0 0" xyz="0 0 0"/>
-      <geometry>
-        <cylinder length="0.02775" radius="0.063"/>
+        <cylinder length="0.02775" radius="0.03625"/>
+      </geometry>
+      <material name="amr_wheel_color"/>
+    </visual>
+    <collision>
+      <origin rpy="1.5707963267949 0 0" xyz="0 0 0"/>
+      <geometry>
+        <cylinder length="0.02775" radius="0.03625"/>
       </geometry>
     </collision>
@@ -216,5 +217,6 @@
     <parent link="amr_main_body"/>
     <child link="left_back_small_wheel"/>
-    <origin rpy="0 0 0" xyz="-0.257 0.2325 -0.022"/>
+    <!-- <origin rpy="0 0 0" xyz="-0.228 0.156 -0.049"/> -->
+    <origin rpy="0 0 0" xyz="-0.257 0.2325 -0.049"/>
   </joint>
   <link name="right_back_small_wheel">
@@ -222,12 +224,12 @@
       <origin rpy="1.5707963267949 0 0" xyz="0 0 0"/>
       <geometry>
-        <cylinder length="0.02775" radius="0.063"/>
-      </geometry>
-      <material name="amr_wheel_color"/>
-    </visual>
-    <collision>
-      <origin rpy="1.5707963267949 0 0" xyz="0 0 0"/>
-      <geometry>
-        <cylinder length="0.02775" radius="0.063"/>
+        <cylinder length="0.02775" radius="0.03625"/>
+      </geometry>
+      <material name="amr_wheel_color"/>
+    </visual>
+    <collision>
+      <origin rpy="1.5707963267949 0 0" xyz="0 0 0"/>
+      <geometry>
+        <cylinder length="0.02775" radius="0.03625"/>
       </geometry>
     </collision>
@@ -241,5 +243,6 @@
     <parent link="amr_main_body"/>
     <child link="right_back_small_wheel"/>
-    <origin rpy="0 0 0" xyz="-0.257 -0.2325 -0.022"/>
+    <!-- <origin rpy="0 0 0" xyz="-0.228 -0.156 -0.049"/> -->
+    <origin rpy="0 0 0" xyz="-0.257 -0.2325 -0.049"/>
   </joint>
 </robot>

Commit message: fixed moma package find issue

File: src/moma_visualisation/urdf/amr_core.xacro (robot description, xacro)
@@ -46,5 +46,5 @@
       <origin rpy="0 0 3.1415926535897" xyz="0 0 -0.085"/>
       <geometry>
-        <mesh filename="package://moma_visualisation/meshes/LD250.obj"/>
+        <mesh filename="file://$(find moma_visualisation)/meshes/LD250.obj"/>
       </geometry>
       <material name="white"/>
